File: STM32F429VET6/STM32F429VET6/Supporting_IC's.sch (KiCad schematic (older format))
At the start: 21 parts

Commit message: Initial Completion of the PDF
Parts:
- added BZ?: Buzzer, Buzzer_Beeper:PUIAudio_SMT_0825_S_4_R, symbol Device:Buzzer
- added C? (x6): 2.2uf/25V, Capacitor_SMD:C_0805_2012Metric_Pad1.15x1.40mm_HandSolder, symbol Device:C_Small
- added C? (x8): 1uf/50V, Capacitor_SMD:C_0805_2012Metric_Pad1.15x1.40mm_HandSolder, symbol Device:C_Small
- added C? (x2): 220uF AL CAP 50V, Capacitor_SMD:CP_Elec_4x4.5, symbol Device:CP1_Small
- added C? (x2): 0.47pf/50V, Capacitor_SMD:C_0805_2012Metric_Pad1.15x1.40mm_HandSolder, symbol Device:C_Small
- added C? (x2): 2.2pf/50V, Capacitor_SMD:C_0805_2012Metric_Pad1.15x1.40mm_HandSolder, symbol Device:C_Small
- added C? (x2): 390pf/50V, Capacitor_SMD:C_0805_2012Metric_Pad1.15x1.40mm_HandSolder, symbol Device:C_Small
- added C? (x2): 1uf/16V, Capacitor_SMD:C_0805_2012Metric_Pad1.15x1.40mm_HandSolder, symbol Device:C_Small
- added C?: 1uf/25V, Capacitor_SMD:C_0805_2012Metric_Pad1.15x1.40mm_HandSolder, symbol Device:C_Small
- added D?: T4, Diode_SMD:D_SOD-123, symbol Diode:1N4148W
- added D?: D, symbol Device:D
- added J? (x2): Conn_01x02, symbol Connector_Generic:Conn_01x02
- added J?: Conn_01x04, symbol Connector_Generic:Conn_01x04
- added J?: Conn_01x20, Connector_FFC-FPC:Hirose_FH12-20S-0.5SH_1x20-1MP_P0.50mm_Horizontal, symbol Connector_Generic:Conn_01x20
- added L? (x2): 10uH, SRN6045TA-100M:SRN6045TA-100M, symbol SRN6045TA-100M:SRN6045TA-100M
- added Q? (x2): BC547-SMD, Package_TO_SOT_SMD:SOT-23, symbol Transistor_BJT:BC547
- added R? (x13): 10K, Resistor_SMD:R_0805_2012Metric_Pad1.15x1.40mm_HandSolder, symbol Device:R_Small
- added R? (x2): 82K, Resistor_SMD:R_0805_2012Metric_Pad1.15x1.40mm_HandSolder, symbol Device:R_Small
- added R? (x2): 10R, Resistor_SMD:R_0805_2012Metric_Pad1.15x1.40mm_HandSolder, symbol Device:R_Small
- added R? (x2): 20K, Resistor_SMD:R_0805_2012Metric_Pad1.15x1.40mm_HandSolder, symbol Device:R_Small
- added R? (x3): 1K, Resistor_SMD:R_0805_2012Metric_Pad1.15x1.40mm_HandSolder, symbol Device:R_Small
- added U?: LM358QT, LM358:LM358QT, symbol LM358:LM358QT
Connections:
- net 24V: now also J?.1 (Pin_1)
- net 3.3V: now also C?.2, C?.2, J?.7 (Pin_7)
- net 5V: now also BZ?.1 (-), C?.1, C?.2, D?.1 (K), R?.2, R?.2, U?.8 (VCC+)
- net BST1: now also C?.2
- net BST2: now also C?.2
- net CH1_INPUT: now also C?.2, R?.2
- net CH2_INPUT: now also C?.2, R?.2
- net GND: now also C?.1, C?.1, C?.1, C?.1, C?.1, C?.1, C?.1, C?.1, C?.1, C?.2, C?.2, C?.2, C?.2, C?.2, D?.2 (A), J?.2 (Pin_2), J?.2 (Pin_2), J?.3 (Pin_3), J?.6 (Pin_6), Q?.3 (E), Q?.3 (E), R?.1, R?.1, R?.1, R?.1, R?.2, R?.2, U?.4 (VCC-), U?.5 (IN2+), U?.6 (IN2-), U?.7 (OUT2)
- net INT1: now also C?.1, C?.2, R?.1, R?.1
- net INT2: now also C?.1, C?.2, R?.1, R?.1
- net SW1: now also C?.1, L?.2, R?.2, R?.2, R?.2
- net SW2: now also C?.1, L?.2, R?.2, R?.2, R?.2
- net TIMER1: now also C?.1
- net TIMER2: now also C?.2
- net at U?.2 (REF1): now also C?.1, C?.1
- net RF2 renamed REF2
- net REF2: now also C?.1, C?.1
- new net: C?.1, R?.2 (x2)
- new net: C?.2, J?.1 (Pin_1) (x2)
- new net: C?.1, C?.2, C?.2, L?.1 (x2)
- new net: C?.2, R?.1 (x2)
- new net: BZ?.2 (+), D?.2 (A), Q?.1 (C)
- new net: Q?.2 (B), R?.1, R?.2 (x2)
- new net: R?.2, R?.2, U?.2 (IN1-)
- new net: C?.2, R?.1, R?.2, U?.3 (IN1+)
- new net: J?.2 (Pin_2), R?.2
- new net: C?.2, J?.4 (Pin_4), R?.1
- new net: C?.1, R?.1
- new net A0: J?.3 (Pin_3)
- new net BUZZER: R?.1
- new net CS1B: J?.1 (Pin_1)
- new net GLCD_LED_CONTROL: R?.1
- new net GLCD_SCLK: J?.4 (Pin_4)
- new net GLCD_SDA: J?.5 (Pin_5)
- new net LED_A: J?.8 (Pin_8), R?.1
- new net LED_K: J?.9 (Pin_9), Q?.1 (C)
- new net MIC_DETECT: C?.1, D?.1 (K), R?.1, R?.2
- new net MIC_OUT: R?.1, R?.1, R?.1, U?.1 (OUT1)
- new net RES: J?.2 (Pin_2)

Commit message: Started working on the ESP32 connection
Parts:
- J?: value Conn_01x20 -> GLCD
Changed lines of the file:
@@
 $Descr A4 11693 8268
 encoding utf-8
-Sheet 3 3
+Sheet 4 4
 Title ""
 Date ""
@@
 P 9600 4750
 F 0 "J?" H 9680 4742 50  0000 L CNN
-F 1 "Conn_01x20" H 9680 4651 50  0000 L CNN
+F 1 "GLCD" H 9680 4651 50  0000 L CNN
 F 2 "Connector_FFC-FPC:Hirose_FH12-20S-0.5SH_1x20-1MP_P0.50mm_Horizontal" H 9600 4750 50  0001 C CNN
 F 3 "~" H 9600 4750 50  0001 C CNN
